File: Electrical/Design/PCBA-KNOT/midi.kicad_sch (KiCad schematic)
At the start: 24 parts, among them U10 BL1551B, U11 BL1551B, U12 6N137, U13 6N137, U14 74HC1G14GV, U9 SESRV05-4

Commit message: SUKU tht jack added
Parts:
- Audio1, Audio2: value PJ-320B -> AUDIO-TH_PJ-3200; footprint suku_basics:AUDIO-SMD_PJ-320B -> suku_basics:AUDIO-TH_PJ-3200
Changed lines of the file:
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@@
 	(label "IN_T"
 		(at 33.02 96.52 0)
-		(fields_autoplaced yes)
 		(effects
 			(font
@@
 	(label "OUT_T"
 		(at 43.18 129.54 90)
-		(fields_autoplaced yes)
 		(effects
 			(font
@@
 	(label "OUT_R"
 		(at 48.26 144.78 270)
-		(fields_autoplaced yes)
 		(effects
 			(font
@@
 	(label "OUT_R"
 		(at 43.18 167.64 0)
-		(fields_autoplaced yes)
 		(effects
 			(font
@@
 	(label "IN_R"
 		(at 58.42 83.82 0)
-		(fields_autoplaced yes)
 		(effects
 			(font
@@
 	(label "OUT_R"
 		(at 33.02 182.88 0)
-		(fields_autoplaced yes)
 		(effects
 			(font
@@
 	(label "IN_R"
 		(at 33.02 99.06 0)
-		(fields_autoplaced yes)
 		(effects
 			(font
@@
 	(label "OUT_T"
 		(at 33.02 180.34 0)
-		(fields_autoplaced yes)
 		(effects
 			(font
@@
 	(label "OUT_T"
 		(at 43.18 165.1 0)
-		(fields_autoplaced yes)
 		(effects
 			(font
@@
 	(label "OUT_T"
 		(at 48.26 129.54 90)
-		(fields_autoplaced yes)
 		(effects
 			(font
@@
 	(label "OUT_R"
 		(at 43.18 144.78 270)
-		(fields_autoplaced yes)
 		(effects
 			(font
@@
 	(label "IN_T"
 		(at 58.42 81.28 0)
-		(fields_autoplaced yes)
 		(effects
 			(font
@@
 		(shape input)
 		(at 116.84 187.96 0)
-		(fields_autoplaced yes)
 		(effects
 			(font
@@
 		(shape output)
 		(at 149.86 96.52 0)
-		(fields_autoplaced yes)
 		(effects
 			(font
@@
 		(shape input)
 		(at 149.86 149.86 0)
-		(fields_autoplaced yes)
 		(effects
 			(font
@@
 			)
 		)
-		(property "Value" "PJ-320B"
+		(property "Value" "AUDIO-TH_PJ-3200"
 			(at 24.13 170.0549 0)
 			(effects
@@
 			)
 		)
-		(property "Footprint" "suku_basics:AUDIO-SMD_PJ-320B"
+		(property "Footprint" "suku_basics:AUDIO-TH_PJ-3200"
 			(at 33.02 157.48 0)
 			(effects
@@
 			)
 		)
-		(property "Value" "PJ-320B"
+		(property "Value" "AUDIO-TH_PJ-3200"
 			(at 38.1 86.2349 0)
 			(effects
@@
 			)
 		)
-		(property "Footprint" "suku_basics:AUDIO-SMD_PJ-320B"
+		(property "Footprint" "suku_basics:AUDIO-TH_PJ-3200"
 			(at 46.99 73.66 0)
 			(effects
